File: Hardware/pianocircuit.brd (EAGLE design)
At the start: 160 x 100 mm, 180 parts

Commit message: Began Board Layout
Parts:
- removed C15, C25, C37, C43, C49, C55: 100n, LinnesLab-Passives:C0603
- removed C16, C17, C18, C19, C20, C26, C27, C28, C29, C30, C38, C39, C40, C41, C42, C44, C45, C46, C47, C48, C50, C51, C52, C53, C54, C56, C57, C58, C59, C60: (no value), LinnesLab-Passives:C0603
- removed OP13, OP14, OP15, OP16, OP17, OP18, OP19, OP20, OP4, OP5, OP7, OP8, OP9: (no value), LinnesLab-AnalogIC:SO8
- removed R18, R24, R25, R31, R32, R38, R39, R40, R41, R60, R61, R62, R63, R69, R70, R71, R72, R78, R79, R80, R81, R87, R88, R89, R90: (no value), LinnesLab-Passives:R0603
- removed R19, R33, R42, R55, R64, R73, R82: 3.3M, LinnesLab-Passives:R0603
- removed R20, R21, R22, R23, R34, R35, R36, R37, R56, R57, R58, R59, R65, R66, R67, R68, R74, R75, R76, R77, R83, R84, R85, R86: 10k, LinnesLab-Passives:R0603
- removed SW10, SW3, SW4, SW5, SW7, SW8, SW9: (no value), LinnesLab-Switches:SPST.KT11P4SM34LFS
- added IC1: LM386M-1, linear:SO08
- added SPK1: (no value), LinnesLab-Electromechanical:SOLDER.TABS
- C10: value (none) -> 330p
- C13: value (none) -> 50n
- C14: value (none) -> 250u; device LinnesLab-Passives:C0603 -> LinnesLab-Passives:C-EEU-FM-A-220UF
- C7: value 100n -> 33n
- C8, C9: value (none) -> 33n
- R10: value 3.3M -> 39k
- R11, R12: value 10k -> 39k
- R15: value (none) -> 390k
- R16: value (none) -> 10k
- R17: device LinnesLab-Passives:R0603 -> LinnesLab-Passives:RTRIMCB10
- moved R49 405.9 mm to (27.9, 14.0)
- moved R50 405.9 mm to (31.8, 14.0)
- moved C31 405.9 mm to (35.6, 31.8)
- moved C32 405.9 mm to (39.4, 22.9)
- moved C33 405.9 mm to (43.2, 22.9)
- moved C34 405.9 mm to (27.9, 17.8)
- moved C35 405.9 mm to (31.8, 17.8)
- moved C36 405.9 mm to (35.6, 17.8)
- moved R43 405.9 mm to (43.2, 31.8)
- moved R44 405.9 mm to (27.9, 22.9)
- moved R45 405.9 mm to (31.8, 22.9)
- moved R46 405.9 mm to (35.6, 22.9)
- moved R47 405.9 mm to (39.4, 17.8)
- moved R48 405.9 mm to (43.2, 17.8)
- moved C14 391.2 mm to (7.62, 91.4)
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Connections:
- removed net N$100: SW9.3, SW9.4
- removed net N$101: OP19.3, R85.1, R86.2
- removed net N$102: C55.2, OP19.1, OP19.2, R84.1
- removed net N$103: OP19.6, R83.1, R84.2
- removed net N$104: C55.1, OP19.5, R82.1
- removed net N$105: OP19.7, R82.2, R83.2, R87.1
- removed net N$106: C57.1, R87.2, R88.1
- removed net N$107: C58.1, R88.2, R89.1
- removed net N$108: C59.1, R89.2, R90.1
- removed net N$109: C60.1, OP20.3, R90.2
- removed net N$110: OP20.1, OP20.2, SW10.1, SW10.2
- removed net N$111: SW10.3, SW10.4
- removed net N$12: SW2.3, SW2.4
- removed net N$13: OP3.3, R13.1, R14.2
- removed net N$18: C9.1, R15.2, R16.1
- removed net N$19: C10.1, R16.2, R17.1
- removed net N$24: OP5.3, R22.1, R23.2
- removed net N$25: C15.2, OP5.1, OP5.2, R21.1
- removed net N$33: OP5.7, R19.2, R20.2, R24.1
- removed net N$34: C17.1, R24.2, R25.1
- removed net N$35: C18.1, R25.2, R31.1
- removed net N$36: C19.1, R31.2, R32.1
- removed net N$37: C20.1, OP7.3, R32.2
- removed net N$38: OP7.1, OP7.2, SW4.1, SW4.2
- removed net N$39: SW4.3, SW4.4
- removed net N$40: OP8.3, R36.1, R37.2
- removed net N$41: C25.2, OP8.1, OP8.2, R35.1
- removed net N$42: OP8.6, R34.1, R35.2
- removed net N$43: C25.1, OP8.5, R33.1
- removed net N$44: OP8.7, R33.2, R34.2, R38.1
- removed net N$45: C27.1, R38.2, R39.1
- removed net N$46: C28.1, R39.2, R40.1
- removed net N$47: C29.1, R40.2, R41.1
- removed net N$48: C30.1, OP9.3, R41.2
- removed net N$49: OP9.1, OP9.2, SW5.1, SW5.2
- removed net N$50: SW5.3, SW5.4
- removed net N$59: SW1.3, SW1.4
- removed net N$67: SW6.3, SW6.4
- removed net N$68: OP13.3, R58.1, R59.2
- removed net N$69: C37.2, OP13.1, OP13.2, R57.1
- removed net N$70: OP13.6, R56.1, R57.2
- removed net N$71: C37.1, OP13.5, R55.1
- removed net N$72: OP13.7, R55.2, R56.2, R60.1
- removed net N$73: C39.1, R60.2, R61.1
- removed net N$74: C40.1, R61.2, R62.1
- removed net N$75: C41.1, R62.2, R63.1
- removed net N$76: C42.1, OP14.3, R63.2
- removed net N$77: OP14.1, OP14.2, SW7.1, SW7.2
- removed net N$78: SW7.3, SW7.4
- removed net N$79: OP15.3, R67.1, R68.2
- removed net N$80: C43.2, OP15.1, OP15.2, R66.1
- removed net N$81: OP15.6, R65.1, R66.2
- removed net N$82: C43.1, OP15.5, R64.1
- removed net N$83: OP15.7, R64.2, R65.2, R69.1
- removed net N$84: C45.1, R69.2, R70.1
- removed net N$85: C46.1, R70.2, R71.1
- removed net N$86: C47.1, R71.2, R72.1
- removed net N$87: C48.1, OP16.3, R72.2
- removed net N$88: OP16.1, OP16.2, SW8.1, SW8.2
- removed net N$89: SW8.3, SW8.4
- removed net N$90: OP17.3, R76.1, R77.2
- removed net N$91: C49.2, OP17.1, OP17.2, R75.1
- removed net N$92: OP17.6, R74.1, R75.2
- removed net N$93: C49.1, OP17.5, R73.1
- removed net N$94: OP17.7, R73.2, R74.2, R78.1
- removed net N$95: C51.1, R78.2, R79.1
- removed net N$96: C52.1, R79.2, R80.1
- removed net N$97: C53.1, R80.2, R81.1
- removed net N$98: C54.1, OP18.3, R81.2
- removed net N$99: OP18.1, OP18.2, SW9.1, SW9.2
- new net A3: R12.2, SW6.3, SW6.4
- new net C3: R10.2, SW2.3, SW2.4
- new net F3: R11.2, SW1.3, SW1.4
- net GND: now also IC1.3, IC1.4, R14.2, R16.1, SPK1.-; no longer C10.2, C13.2, C14.2, C17.2, C18.2, C19.2, C20.2, C27.2, C28.2, C29.2, C30.2, C39.2, C40.2, C41.2, C42.2, C45.2, C46.2, C47.2, C48.2, C51.2, C52.2, C53.2, C54.2, C57.2, C58.2, C59.2, C60.2, C9.2, OP13.4, OP15.4, OP17.4, OP19.4, OP3.4, OP5.4, OP8.4, R14.1, R23.1, R37.1, R59.1, R68.1, R77.1, R86.1
- net N$14: now also R10.1; no longer OP3.1, OP3.2, R12.1
- net N$15: now also C10.2, C7.1, C8.1, C9.1, OP3.3, R15.2; no longer OP3.6, R11.1, R12.2
- net N$16: now also C9.2, R12.1; no longer C7.1, OP3.5, R10.1
- net N$17: now also C8.2, R11.1; no longer OP3.7, R10.2, R11.2, R15.1
- net N$2: no longer C16.1, C26.1, C38.1, C44.1, C50.1, C56.1, C8.1
- net N$20: now also C10.1, OP3.1, R15.1, R17.C; no longer C13.1, R17.2, R18.1
- net N$21: now also OP3.2, R13.1, R14.1; no longer C14.1, OP4.3, R18.2
- net N$22: now also IC1.2, R17.B; no longer OP4.1, OP4.2, SW3.1, SW3.2
- net N$23: now also C13.2, R16.2; no longer SW3.3, SW3.4
- net N$26: now also C13.1, C14.+, IC1.5; no longer OP5.6, R20.1, R21.2
- net N$32: now also C14.-, SPK1.+; no longer C15.1, OP5.5, R19.1
- net N$60: no longer R42.1
- net N$61: no longer R42.2
- net V+: now also OP3.8; no longer OP14.8, OP16.8, OP18.8, OP20.8, OP4.8, OP7.8, OP9.8
- net V-: now also OP3.4; no longer OP14.4, OP16.4, OP18.4, OP20.4, OP4.4, OP7.4, OP9.4
- net V_BATT: now also IC1.6; no longer C16.2, C26.2, C38.2, C44.2, C50.2, C56.2, C8.2, OP13.8, OP15.8, OP17.8, OP19.8, OP3.8, OP5.8, OP8.8, R22.2, R36.2, R58.2, R67.2, R76.2, R85.2

Commit message: Board Routing
Parts:
- moved OP12 69.9 mm to (92.7, 40.6), turned to 270 degrees
- moved SW6 67.9 mm to (52.1, 68.6)
- moved R11 67.9 mm to (87.6, 62.2)
- moved OP3 66.0 mm to (68.6, 40.6), turned to 270 degrees
- moved R10 53.4 mm to (69.8, 62.2)
- moved C9 51.1 mm to (58.4, 54.6)
- moved R14 48.8 mm to (61.0, 36.8)
- moved C10 46.6 mm to (58.4, 41.9), turned to 270 degrees
- moved C21 46.4 mm to (72.4, 2.54)
- moved SW1 43.2 mm to (147.3, 71.1)
- moved SW2 41.3 mm to (100.3, 69.8)
- moved R12 38.7 mm to (58.4, 62.2), turned to 180 degrees
- moved R52 37.0 mm to (81.3, 2.54)
- moved R13 36.7 mm to (31.8, 36.8)
- moved R15 36.6 mm to (53.3, 41.9), turned to 270 degrees
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Routing:
- net N$14: track 0.00 -> 113.9 mm
- net N$28: track 0.00 -> 97.8 mm
- net N$10: track 0.00 -> 92.7 mm
- net N$54: track 0.00 -> 88.8 mm
- net N$55: track 0.00 -> 85.5 mm
- net N$65: track 0.00 -> 85.1 mm
- net N$17: track 0.00 -> 81.1 mm
- net N$15: track 0.00 -> 79.9 mm
- net N$20: track 0.00 -> 62.7 mm
- net N$66: track 0.00 -> 54.4 mm
- net N$58: track 0.00 -> 47.0 mm
- net N$2: track 0.00 -> 43.5 mm
- net N$11: track 0.00 -> 43.0 mm
- net N$7: track 0.00 -> 43.0 mm
- net N$57: track 0.00 -> 40.7 mm
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Other:
- board size 160 x 100 mm -> 160 x 82.2 mm

Commit message: Updated Board Routing
Routing:
- net F3: track 0.00 -> 107.6 mm
Changed lines of the file:
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@@
 <drawing>
 <settings>
-<setting alwaysvectorfont="yes"/>
+<setting alwaysvectorfont="no"/>
 <setting verticaltext="up"/>
 </settings>
@@
 <contactref element="SW1" pad="4"/>
 <contactref element="SW1" pad="3"/>
-<wire x1="151.4475" y1="69.1" x2="143.1925" y2="69.1" width="0" layer="19" extent="1-1"/>
-<wire x1="88.48" y1="62.23" x2="143.1925" y2="69.1" width="0" layer="19" extent="1-1"/>
+<wire x1="141.6314" y1="72.2503125" x2="141.6314" y2="74.0296875" width="0.1524" layer="1"/>
+<wire x1="141.6314" y1="74.0296875" x2="141.7653125" y2="74.1636" width="0.1524" layer="1"/>
+<wire x1="152.8746875" y1="74.1636" x2="153.0086" y2="74.0296875" width="0.1524" layer="1"/>
+<wire x1="153.0086" y1="74.0296875" x2="153.0086" y2="72.2503125" width="0.1524" layer="1"/>
+<wire x1="143.1925" y1="69.1" x2="143.1925" y2="70.6892125" width="0.1524" layer="1"/>
+<wire x1="143.1925" y1="70.6892125" x2="141.6314" y2="72.2503125" width="0.1524" layer="1"/>
+<wire x1="141.7653125" y1="74.1636" x2="152.8746875" y2="74.1636" width="0.1524" layer="1"/>
+<wire x1="153.0086" y1="72.2503125" x2="152.4" y2="71.6417125" width="0.1524" layer="1"/>
+<wire x1="152.4" y1="71.6417125" x2="152.4" y2="69.85" width="0.1524" layer="1"/>
+<wire x1="94.7753125" y1="70.8464" x2="94.6414" y2="70.9803125" width="0.1524" layer="1"/>
+<wire x1="94.6414" y1="70.9803125" x2="94.6414" y2="72.7596875" width="0.1524" layer="1"/>
+<wire x1="94.6414" y1="72.7596875" x2="94.7753125" y2="72.8936" width="0.1524" layer="1"/>
+<wire x1="88.48" y1="62.23" x2="101.3082875" y2="62.23" width="0.1524" layer="1"/>
+<wire x1="101.3082875" y1="62.23" x2="106.0186" y2="66.9403125" width="0.1524" layer="1"/>
+<wire x1="106.0186" y1="66.9403125" x2="106.0186" y2="68.7196875" width="0.1524" layer="1"/>
+<wire x1="106.0186" y1="68.7196875" x2="103.8918875" y2="70.8464" width="0.1524" layer="1"/>
+<wire x1="125.6586" y1="70.4446875" x2="125.6586" y2="69.3981125" width="0.1524" layer="1"/>
+<wire x1="125.6586" y1="69.3981125" x2="125.9567125" y2="69.1" width="0.1524" layer="1"/>
+<wire x1="125.9567125" y1="69.1" x2="143.1925" y2="69.1" width="0.1524" layer="1"/>
+<wire x1="103.8918875" y1="70.8464" x2="94.7753125" y2="70.8464" width="0.1524" layer="1"/>
+<wire x1="94.7753125" y1="72.8936" x2="123.2096875" y2="72.8936" width="0.1524" layer="1"/>
+<wire x1="123.2096875" y1="72.8936" x2="125.6586" y2="70.4446875" width="0.1524" layer="1"/>
+<wire x1="152.4" y1="69.85" x2="151.4475" y2="69.1" width="0" layer="19" extent="1-1"/>
 </signal>
 <signal name="A3">

Commit message: Reorganizing Board
Parts:
- moved C7 72.7 mm to (114.3, 57.1)
- moved C8 55.8 mm to (86.4, 57.1), turned to 180 degrees
- moved R15 51.2 mm to (90.2, 77.5), turned to 0 degrees
- moved C5 46.2 mm to (154.9, 8.89)
- moved R10 45.8 mm to (115.6, 64.8)
- moved SW1 45.7 mm to (101.6, 69.8)
- moved R17 45.4 mm to (25.4, 73.7), turned to 90 degrees
- moved SW2 44.5 mm to (144.8, 71.1)
- moved C10 44.0 mm to (90.2, 72.4), turned to 0 degrees
- moved OP11 38.1 mm to (109.2, 40.6)
- moved C23 37.6 mm to (118.1, 33.0)
- moved R9 36.9 mm to (157.5, 5.08)
- moved R27 33.0 mm to (95.2, 20.3)
- moved R8 32.1 mm to (157.5, 12.7), turned to 180 degrees
- moved R28 29.6 mm to (91.4, 20.3)
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Routing:
- net N$14: track 113.9 -> 0.00 mm
- net F3: track 107.6 -> 0.00 mm
- net N$28: track 97.8 -> 0.00 mm
- net N$10: track 92.7 -> 0.00 mm
- net N$54: track 88.8 -> 0.00 mm
- net N$65: track 85.1 -> 0.00 mm
- net N$55: track 85.5 -> 1.00 mm
- net N$17: track 81.1 -> 0.00 mm
- net N$15: track 79.9 -> 0.00 mm
- net N$20: track 62.7 -> 0.30 mm
- net N$66: track 54.4 -> 0.00 mm
- net N$58: track 47.0 -> 0.30 mm
- net N$2: track 43.5 -> 0.00 mm
- net N$11: track 43.0 -> 0.00 mm
- net N$7: track 43.0 -> 0.00 mm
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
Commit message: Reorganized
Parts:
- moved C21 10.9 mm to (101.6, 15.2)
- moved C11 9.16 mm to (86.4, 8.89), turned to 180 degrees
- moved R28 6.35 mm to (85.1, 20.3)
- moved R52 5.24 mm to (101.6, 17.8)
- moved C32 5.08 mm to (54.6, 24.1)
- moved R27 5.08 mm to (90.2, 20.3)
- moved R26 3.59 mm to (95.2, 20.3), turned to 180 degrees
- moved R53 3.59 mm to (99.1, 11.4)
- moved R51 2.54 mm to (101.6, 20.3), turned to 0 degrees
- moved R54 1.27 mm to (101.6, 8.89)
Routing:
- net N$26: track 0.33 -> 19.0 mm
- net N$32: track 0.00 -> 16.1 mm

Commit message: Updated Schematic
Parts:
- removed C2, C32: (no value), LinnesLab-Passives:C0603
- removed R4, R45, R46, R5: 10k, LinnesLab-Passives:R0603
Connections:
- removed net N$1: OP1.3, R4.1, R5.2
- removed net N$28: C11.2, OP6.1, OP6.2, R28.1
- removed net N$51: OP10.3, R45.1, R46.2
- removed net N$56: C31.2, OP10.1, OP10.2, R44.1
- net GND: no longer OP1.4, OP10.4, R46.1, R5.1
- net N$2: no longer C2.1, C32.1
- net N$3: now also C11.2, C31.2, OP6.1, OP6.2, R28.1, R44.1; no longer OP1.1, OP1.2
- net V+: now also OP1.8, OP10.8
- net V-: now also OP1.4, OP10.4
- net V_BATT: no longer C2.2, C32.2, OP1.8, OP10.8, R4.2, R45.2
Routing:
- net N$56: track 1.35 -> 0.00 mm
- net N$3: track 0.00 -> 0.65 mm

Commit message: Updated Board Routing
Parts:
- moved R10 17.0 mm to (130.8, 57.1)
- moved OP10 11.4 mm to (30.5, 24.1)
- moved C1 10.2 mm to (141.0, 7.62), turned to 180 degrees
- moved C9 10.2 mm to (68.6, 55.9), turned to 180 degrees
- moved R54 5.68 mm to (106.7, 11.4)
- moved R2 5.24 mm to (148.6, 17.8)
- moved R29 5.08 mm to (78.7, 20.3)
- moved R3 5.08 mm to (141.0, 17.8)
- moved C21 4.58 mm to (105.4, 17.8), turned to 0 degrees
- moved C5 2.84 mm to (152.4, 7.62)
- moved R30 2.54 mm to (78.7, 14.0)
- moved R53 2.54 mm to (101.6, 11.4)
- moved R28 1.80 mm to (86.4, 21.6)
- moved C8 1.80 mm to (85.1, 55.9)
- moved R6 1.27 mm to (151.1, 22.9)
Routing:
- net N$3: track 0.65 -> 148.7 mm
- net N$15: track 0.00 -> 118.8 mm
- net N$20: track 0.30 -> 103.9 mm
- net N$11: track 0.00 -> 50.6 mm
- net N$66: track 0.00 -> 49.6 mm
- net N$55: track 1.00 -> 50.4 mm
- net N$57: track 0.00 -> 45.5 mm
- net N$10: track 0.00 -> 39.0 mm
- net N$63: track 1.29 -> 36.2 mm
- net N$26: track 19.0 -> 49.6 mm
- net N$54: track 0.00 -> 30.0 mm
- net V+: track 0.00 -> 28.8 mm
- net N$62: track 0.00 -> 27.9 mm
- net C3: track 0.00 -> 23.9 mm
- net N$22: track 0.00 -> 22.6 mm
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
Commit message: Updated Routing
Connections:
- removed net V+: OP1.8, OP10.8, OP11.8, OP12.8, OP2.8, OP3.8
- removed net V-: OP1.4, OP10.4, OP11.4, OP12.4, OP2.4, OP3.4
- removed net V_BATT: C12.2, IC1.6, OP6.8, R13.2, R29.2
- new net 5V: C12.2, IC1.6, OP1.8, OP10.8, OP11.8, OP12.8, OP2.8, OP3.8, OP6.8, R13.2, R29.2
- net GND: now also OP1.4, OP10.4, OP11.4, OP12.4, OP2.4, OP3.4
Routing:
- net N$65: track 16.9 -> 88.6 mm
- net N$61: track 11.9 -> 64.4 mm
- net V+: track 28.8 -> 0.00 mm
- net 5V: track 0.00 -> 28.8 mm
- net GND: track 0.00 -> 28.0 mm, vias 0 -> 21
- net N$58: track 17.6 -> 33.3 mm
- added copper zone on layer 1, net 5V
- added copper zone on layer 16, net GND
